File: Kicad/Eve/Robourt.kicad_pcb (KiCad board)
At the start: 4 copper layers, 85 x 67.1 mm, 172 parts, among them IC101 STM32U535RET6, J1 Conn_02x08_Odd_Even, J101 Conn_ST_STDC14, J102 Conn_01x02, J103 Conn_01x02, J108 Conn_01x03, J109 Conn_01x03, J110 Conn_01x02, J115 Conn_02x20_Odd_Even, J201 Conn_01x04, J301 Conn_01x04, J401 Conn_01x04, Q101 NMOS, Q201 SQJ504EP-T1_GE3, Q202 SQJ504EP-T1_GE3, Q203 SQJ504EP-T1_GE3, Q204 SQJ504EP-T1_GE3, Q301 SQJ504EP-T1_GE3, Q302 SQJ504EP-T1_GE3, Q303 SQJ504EP-T1_GE3, Q304 SQJ504EP-T1_GE3, Q401 SQJ504EP-T1_GE3, Q402 SQJ504EP-T1_GE3, Q403 SQJ504EP-T1_GE3, Q404 SQJ504EP-T1_GE3, SW101 SW_Push, SW102 SW_Push, SW103 SW_Push, SW104 SW_Push, U201 TMC2590-TA, U301 TMC2590-TA, U401 TMC2590-TA, U501 BU33SD5WG-TR, U601 LT1076CR-PBF, U701 LT1076CR-PBF, U801 LT1076CR-PBF, Y101 Crystal

Commit message: update pcb
Parts:
- removed Q201, Q202, Q203, Q204, Q301, Q302, Q303, Q304, Q401, Q402, Q403, Q404: SQJ504EP-T1_GE3, Mosfet:SQJ968EPT1GE3
- removed R201, R202, R301, R302, R401, R402: 0.075, Resistor_SMD:R_2512_6332Metric
- removed R203, R204, R303, R304, R403, R404: 10, Resistor_SMD:R_0402_1005Metric
- added R1: 75m, Resistor_SMD:R_2512_6332Metric, B.Cu at (106.1, -3.76)
- added R10: 10, Resistor_SMD:R_0402_1005Metric, B.Cu at (72.9, -28.4)
- added R11: 75m, Resistor_SMD:R_2512_6332Metric, B.Cu at (39.8, 27.0)
- added R12: 10, Resistor_SMD:R_0402_1005Metric, B.Cu at (30.1, 43.6)
- added R2: 75m, Resistor_SMD:R_2512_6332Metric, B.Cu at (67.1, -28.9)
- added R3: 75m, Resistor_SMD:R_2512_6332Metric, B.Cu at (46.3, 42.8)
- added R4: 10, Resistor_SMD:R_0402_1005Metric, B.Cu at (111.9, -5.21)
- added R5: 10, Resistor_SMD:R_0402_1005Metric, B.Cu at (72.9, -30.4)
- added R6: 10, Resistor_SMD:R_0402_1005Metric, B.Cu at (39.8, 43.2)
- added R7: 75m, Resistor_SMD:R_2512_6332Metric, B.Cu at (106.1, 1.13)
- added R8: 10, Resistor_SMD:R_0402_1005Metric, B.Cu at (111.9, -3.22)
- added R9: 75m, Resistor_SMD:R_2512_6332Metric, B.Cu at (67.1, -24.0)
- added U1: SQJ504EP-T1, Mosfet:SQJ968EPT1GE3, F.Cu at (89.1, 45.8)
- added U10: SQJ504EP-T1, Mosfet:SQJ968EPT1GE3, F.Cu at (71.9, 22.6)
- added U11: SQJ504EP-T1, Mosfet:SQJ968EPT1GE3, F.Cu at (43.4, 22.6)
- added U12: SQJ504EP-T1, Mosfet:SQJ968EPT1GE3, F.Cu at (49.2, 22.6)
- added U2: SQJ504EP-T1, Mosfet:SQJ968EPT1GE3, F.Cu at (66.3, 45.8)
- added U3: SQJ504EP-T1, Mosfet:SQJ968EPT1GE3, F.Cu at (43.5, 45.8)
- added U4: SQJ504EP-T1, Mosfet:SQJ968EPT1GE3, F.Cu at (94.8, 45.8)
- added U5: SQJ504EP-T1, Mosfet:SQJ968EPT1GE3, F.Cu at (72.1, 45.8)
- added U6: SQJ504EP-T1, Mosfet:SQJ968EPT1GE3, F.Cu at (49.3, 45.8)
- added U7: SQJ504EP-T1, Mosfet:SQJ968EPT1GE3, F.Cu at (88.8, 22.7)
- added U8: SQJ504EP-T1, Mosfet:SQJ968EPT1GE3, F.Cu at (94.6, 22.7)
- added U9: SQJ504EP-T1, Mosfet:SQJ968EPT1GE3, F.Cu at (66.1, 22.6)
- moved C401 2.01 mm to (47.0, 21.2), turned to 90 degrees
- moved R124 0.30 mm to (85.7, 78.5)
- moved C116 0.30 mm to (85.7, 79.5)
- moved C106 0.15 mm to (85.9, 80.8)
Connections:
- U601 pad 8: GND1 -> (no net)
- U701 pad 8: GND1 -> (no net)
- U801 pad 8: GND1 -> (no net)
Routing:
- net +3.3V: track 54.9 -> 123.7 mm
- net /driver_stepper2/LS_Gnd: track 0.00 -> 26.4 mm, vias 0 -> 18
- net /driver_stepper2/SRB: track 23.6 -> 2.13 mm, vias 2 -> 0
- net /driver_stepper1/S: track 17.6 -> 0.00 mm, vias 2 -> 0
- net /driver_stepper2/S: track 17.6 -> 0.00 mm, vias 2 -> 0
- net /driver_stepper/S: track 17.5 -> 0.00 mm, vias 2 -> 0
- net Net-(R1-Pad2): track 0.00 -> 14.5 mm, vias 0 -> 2
- net Net-(Q201-S1): track 14.5 -> 0.00 mm, vias 2 -> 0
- net Net-(R3-Pad2): track 0.00 -> 14.4 mm, vias 0 -> 2
- net Net-(Q401-S1): track 14.4 -> 0.00 mm, vias 2 -> 0
- net Net-(R2-Pad2): track 0.00 -> 14.3 mm, vias 0 -> 2
- net Net-(Q301-S1): track 14.3 -> 0.00 mm, vias 2 -> 0
- net /driver_stepper2/LB1: track 35.7 -> 25.8 mm
- net (no net): track 0.00 -> 7.04 mm, vias 0 -> 4
- net GND1: track 127.2 -> 122.6 mm, vias 565 -> 563
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- added copper zone on B.Cu, net /driver_stepper2/LS_Gnd
- added copper zone on F.Cu, net /driver_stepper2/LS_Gnd
- added copper zone on In2.Cu, net 24V
- added copper zone on In1.Cu, net GND1
