File: Kicad/Eve/Robourt.kicad_sch (KiCad schematic)
At the start: 77 parts, among them IC101 STM32U535RET6, J1 Conn_02x08_Odd_Even, J102 Conn_01x02, J103 Conn_01x02, J108 Conn_01x03, J109 Conn_01x03, J110 Conn_01x02, Q101 NMOS, Y101 Crystal

Commit message: update pcb
Parts:
- renumbered J1 to J104, J108 to J105, J109 to J106, J110 to J107
Changed lines of the file:
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@@
       (project "Robourt"
         (path "/87ede840-4957-4951-b25a-c132e7988ddc"
-          (reference "J115") (unit 1)
+          (reference "J108") (unit 1)
         )
       )
@@
           (reference "#PWR0146") (unit 1)
         )
-        (path "/87ede840-4957-4951-b25a-c132e7988ddc/b0f3c6bf-43ee-43a7-9a34-92e1e933f121"
-          (reference "#PWR?") (unit 1)
-        )
       )
     )
@@
   (symbol (lib_id "Connector_Generic:Conn_01x03") (at 243.84 129.54 0) (unit 1)
     (in_bom yes) (on_board yes) (dnp no) (fields_autoplaced)
-    (property "Reference" "J109" (at 246.38 128.905 0)
+    (property "Reference" "J106" (at 246.38 128.905 0)
       (effects (font (size 1.27 1.27)) (justify left))
     )
@@
       (project "Robourt"
         (path "/87ede840-4957-4951-b25a-c132e7988ddc"
-          (reference "J109") (unit 1)
-        )
-        (path "/87ede840-4957-4951-b25a-c132e7988ddc/c08e9c7d-1604-43bb-a00c-546e3bb44d34"
-          (reference "J?") (unit 1)
+          (reference "J106") (unit 1)
         )
       )
@@
           (reference "#PWR0147") (unit 1)
         )
-        (path "/87ede840-4957-4951-b25a-c132e7988ddc/c08e9c7d-1604-43bb-a00c-546e3bb44d34"
-          (reference "#PWR?") (unit 1)
-        )
       )
     )
@@
   (symbol (lib_id "Connector_Generic:Conn_02x08_Odd_Even") (at 228.6 160.02 0) (unit 1)
     (in_bom yes) (on_board yes) (dnp no) (fields_autoplaced)
-    (property "Reference" "J1" (at 229.87 146.05 0)
+    (property "Reference" "J104" (at 229.87 146.05 0)
       (effects (font (size 1.27 1.27)))
     )
@@
       (project "Robourt"
         (path "/87ede840-4957-4951-b25a-c132e7988ddc"
-          (reference "J1") (unit 1)
+          (reference "J104") (unit 1)
         )
       )
@@
   (symbol (lib_id "Connector_Generic:Conn_01x03") (at 243.84 113.03 0) (unit 1)
     (in_bom yes) (on_board yes) (dnp no)
-    (property "Reference" "J108" (at 246.38 112.395 0)
+    (property "Reference" "J105" (at 246.38 112.395 0)
       (effects (font (size 1.27 1.27)) (justify left))
     )
@@
       (project "Robourt"
         (path "/87ede840-4957-4951-b25a-c132e7988ddc"
-          (reference "J108") (unit 1)
-        )
-        (path "/87ede840-4957-4951-b25a-c132e7988ddc/b0f3c6bf-43ee-43a7-9a34-92e1e933f121"
-          (reference "J?") (unit 1)
+          (reference "J105") (unit 1)
         )
       )
@@
   (symbol (lib_id "Connector_Generic:Conn_01x02") (at 250.19 92.71 0) (mirror x) (unit 1)
     (in_bom yes) (on_board yes) (dnp no) (fields_autoplaced)
-    (property "Reference" "J110" (at 250.19 85.09 0)
+    (property "Reference" "J107" (at 250.19 85.09 0)
       (effects (font (size 1.27 1.27)))
     )
@@
       (project "Robourt"
         (path "/87ede840-4957-4951-b25a-c132e7988ddc"
-          (reference "J110") (unit 1)
+          (reference "J107") (unit 1)
         )
       )
