File: Kicad/Eve/driver_stepper.kicad_sch (KiCad schematic)
At the start: 19 parts, among them J201 Conn_01x04, Q201 SQJ504EP-T1_GE3, Q202 SQJ504EP-T1_GE3, Q203 SQJ504EP-T1_GE3, Q204 SQJ504EP-T1_GE3, U201 TMC2590-TA

Commit message: update pcb
Parts:
- removed Q201, Q202, Q203, Q204: SQJ504EP-T1_GE3, Mosfet:SQJ968EPT1GE3, symbol SQJ504EP-T1_GE3:SQJ504EP-T1_GE3
- removed R201, R202: 0.075, Resistor_SMD:R_2512_6332Metric, symbol Device:R
- removed R203, R204: 10, Resistor_SMD:R_0402_1005Metric, symbol Device:R
- added R1, R7: 75m, Resistor_SMD:R_2512_6332Metric, symbol Device:R
- added R4, R8: 10, Resistor_SMD:R_0402_1005Metric, symbol Device:R
- added U1, U4, U7, U8: SQJ504EP-T1, Mosfet:SQJ968EPT1GE3, symbol SQJ504EP-T1:SQJ504EP-T1_GE3
Connections:
- net A1: now also U1.5 (D), U1.6 (D)
- net A2: now also U4.5 (D), U4.6 (D)
- net B1: now also U7.5 (D), U7.6 (D)
- net B2: now also U8.5 (D), U8.6 (D)
- net GND: now also R1.1, R7.1
- net HA1: now also U1.4 (G)
- net HA2: now also U4.4 (G)
- net HB1: now also U7.4 (G)
- net HB2: now also U8.4 (G)
- net LA1: now also U1.2 (G)
- net LA2: now also U4.2 (G)
- net LB1: now also U7.2 (G)
- net LB2: now also U8.2 (G)
- net SRA: now also R4.2
- net SRB: now also R8.2
- net Vdc: now also U1.3 (S), U4.3 (S), U7.3 (S), U8.3 (S)
- new net: R1.2, R4.1, U1.1 (S), U4.1 (S)
- new net LS_Gnd: R7.2, R8.1, U7.1 (S), U8.1 (S)

Commit message: update pcb
Parts:
- added C202: 100n, Capacitor_SMD:C_0402_1005Metric, symbol Device:C_Small
- added C205: 10u, Capacitor_SMD:C_2220_5750Metric, symbol Device:C_Small
- added R204, R206: 0, Custom:Wire_Shunt_Kelvin, symbol Device:R
- renumbered C202 to C203, C203 to C204, C204 to C206, C205 to C207, C206 to C208, C207 to C209, C208 to C210, C209 to C211, R1 to R201, R7 to R202, R4 to R203, R8 to R205, U1 to U202, U7 to U203, U4 to U204, U8 to U205
Connections:
- net GND: now also C202.2, C205.2, R204.1, R206.1; no longer U201.13 (SRBL), U201.28 (SRAL)
- net Vdc: now also C202.1, C205.1
- net LS_A: now reaches R201.2, R203.1, U202.1 (S), U204.1 (S)
- net LS_Gnd renamed LS_B
- new net SRAL: R204.2, U201.28 (SRAL)
- new net SRBL: R206.2, U201.13 (SRBL)
Other:
- moved on the sheet: C206, C207
