File: Kicad/Eve/untitled.kicad_sch (KiCad schematic)
At the start: 5 parts, among them U501 BU33SD5WG-TR

Commit message: update pcb
Parts:
- gave numbers to parts that had none: 2
Changed lines of the file:
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@@
   (symbol (lib_id "Device:LED") (at 209.55 87.63 90) (unit 1)
     (in_bom yes) (on_board yes) (dnp no) (fields_autoplaced)
-    (property "Reference" "D?" (at 213.36 88.5825 90)
+    (property "Reference" "D501" (at 213.36 88.5825 90)
       (effects (font (size 1.27 1.27)) (justify right))
     )
@@
     (instances
       (project "Robourt"
-        (path "/87ede840-4957-4951-b25a-c132e7988ddc"
-          (reference "D?") (unit 1)
-        )
         (path "/87ede840-4957-4951-b25a-c132e7988ddc/45a40ff7-b6ec-4165-9635-bd80258dd043"
           (reference "D501") (unit 1)
@@
   (symbol (lib_id "Device:R_Small") (at 209.55 77.47 0) (unit 1)
     (in_bom yes) (on_board yes) (dnp no) (fields_autoplaced)
-    (property "Reference" "R?" (at 212.09 76.835 0)
+    (property "Reference" "R501" (at 212.09 76.835 0)
       (effects (font (size 1.27 1.27)) (justify left))
     )
@@
     (instances
       (project "Robourt"
-        (path "/87ede840-4957-4951-b25a-c132e7988ddc"
-          (reference "R?") (unit 1)
-        )
         (path "/87ede840-4957-4951-b25a-c132e7988ddc/45a40ff7-b6ec-4165-9635-bd80258dd043"
           (reference "R501") (unit 1)
@@
   (symbol (lib_id "power:GND") (at 209.55 97.79 0) (unit 1)
     (in_bom yes) (on_board yes) (dnp no) (fields_autoplaced)
-    (property "Reference" "#PWR?" (at 209.55 104.14 0)
+    (property "Reference" "#PWR0502" (at 209.55 104.14 0)
       (effects (font (size 1.27 1.27)) hide)
     )
@@
     (instances
       (project "Robourt"
-        (path "/87ede840-4957-4951-b25a-c132e7988ddc"
-          (reference "#PWR?") (unit 1)
-        )
         (path "/87ede840-4957-4951-b25a-c132e7988ddc/45a40ff7-b6ec-4165-9635-bd80258dd043"
           (reference "#PWR0502") (unit 1)
